File: Macro14 PCB/Macro14 PCB.kicad_pcb (KiCad board)
At the start: 2 copper layers, 15 parts, among them SW1 Rotary_Encoder_Switch, SW2 Rotary_Encoder_Switch, U1 Pico

Commit message: PCB completed and schematic updated
Parts:
- added REF**: MountingHole_3.2mm_M3, MountingHole:MountingHole_3.2mm_M3, F.Cu at (195.0, -50.0)
- added REF**: MountingHole_3.2mm_M3, MountingHole:MountingHole_3.2mm_M3, F.Cu at (195.0, -5.00)
- added REF**: MountingHole_3.2mm_M3, MountingHole:MountingHole_3.2mm_M3, F.Cu at (105.0, -5.00)
- added REF**: MountingHole_3.2mm_M3, MountingHole:MountingHole_3.2mm_M3, F.Cu at (105.0, -95.0)
- U1: moved to B.Cu
- moved SW2 150.7 mm to (138.0, -71.0)
- moved MX5 134.4 mm to (121.5, -40.5)
- moved MX6 134.4 mm to (140.5, -40.5)
- moved MX7 134.4 mm to (159.5, -40.5)
- moved MX8 134.4 mm to (178.5, -40.5)
- moved MX1 134.4 mm to (121.5, -59.5)
- moved MX10 134.4 mm to (140.5, -21.5)
- moved MX11 134.4 mm to (159.5, -21.5)
- moved MX2 134.4 mm to (140.5, -59.5)
- moved MX3 134.4 mm to (159.5, -59.5)
- moved MX4 134.4 mm to (178.5, -59.5)
- moved MX9 134.4 mm to (121.5, -21.5)
- moved SW1 118.7 mm to (119.0, -71.0)
- moved U1 101.8 mm to (174.0, -84.5), turned to 90 degrees
- moved MX12 13.4 mm to (178.5, -21.5)
Connections:
- U1 pad 10: Net-(MX2-Pad2) -> Net-(MX1-Pad2)
- U1 pad 11: Net-(MX1-Pad2) -> Net-(MX8-Pad2)
- U1 pad 12: Net-(MX8-Pad2) -> Net-(MX7-Pad2)
- U1 pad 14: Net-(MX7-Pad2) -> Net-(MX6-Pad2)
- U1 pad 15: Net-(MX6-Pad2) -> Net-(MX5-Pad2)
- U1 pad 16: Net-(MX5-Pad2) -> Net-(MX12-Pad2)
- U1 pad 17: Net-(MX12-Pad2) -> Net-(MX11-Pad2)
- U1 pad 19: Net-(MX11-Pad2) -> Net-(MX10-Pad2)
- U1 pad 2: Net-(SW2-PadB) -> Net-(U1-Pad2)
- U1 pad 20: Net-(MX10-Pad2) -> Net-(MX9-Pad2)
- U1 pad 21: Net-(MX9-Pad2) -> Net-(SW1-PadS1)
- U1 pad 22: Net-(U1-Pad22) -> Net-(SW2-PadS1)
- U1 pad 24: Net-(SW2-PadS1) -> Net-(SW2-PadB)
- U1 pad 25: Net-(U1-Pad25) -> Net-(SW2-PadA)
- U1 pad 26: Net-(U1-Pad26) -> Net-(SW1-PadB)
- U1 pad 27: Net-(U1-Pad27) -> Net-(SW1-PadA)
- U1 pad 33: Net-(U1-Pad33) -> GND
- U1 pad 4: Net-(SW2-PadA) -> Net-(U1-Pad4)
- U1 pad 42: Net-(U1-Pad42) -> GND
- U1 pad 5: Net-(SW1-PadB) -> Net-(U1-Pad5)
- U1 pad 6: Net-(SW1-PadA) -> Net-(MX4-Pad2)
- U1 pad 7: Net-(MX4-Pad2) -> Net-(MX3-Pad2)
- U1 pad 9: Net-(MX3-Pad2) -> Net-(MX2-Pad2)
Routing:
- net Net-(MX9-Pad2): track 0.00 -> 240.2 mm
- net Net-(MX10-Pad2): track 0.00 -> 220.6 mm
- net Net-(MX11-Pad2): track 0.00 -> 203.6 mm
- net Net-(MX12-Pad2): track 0.00 -> 182.7 mm
- net Net-(MX1-Pad2): track 0.00 -> 61.0 mm
- net Net-(SW1-PadA): track 0.00 -> 58.6 mm, vias 0 -> 1
- net Net-(MX5-Pad2): track 0.00 -> 55.8 mm
- net Net-(SW1-PadB): track 0.00 -> 53.2 mm, vias 0 -> 1
- net Net-(MX6-Pad2): track 0.00 -> 48.3 mm
- net Net-(MX2-Pad2): track 0.00 -> 44.6 mm
- net Net-(SW2-PadA): track 0.00 -> 39.0 mm
- net Net-(MX7-Pad2): track 0.00 -> 34.1 mm
- net Net-(MX8-Pad2): track 0.00 -> 34.1 mm
- net Net-(SW2-PadB): track 0.00 -> 33.4 mm
- net Net-(SW1-PadS1): track 0.00 -> 29.1 mm
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- added copper zone on B.Cu, net GND
Other:
- board outline added: 100 x 100 mm
