File: Macro14 PCB/Macro14 PCB.sch (KiCad schematic (older format))
At the start: 15 parts

Commit message: Finished Schematic
Parts:
- MX1, MX10, MX11, MX12, MX2, MX3, MX4, MX5, MX6, MX7, MX8, MX9: renamed from MX?; footprint (none) -> MX_Only:MXOnly-1U-NoLED
- SW1, SW2: renamed from SW?; footprint (none) -> Rotary_Encoder:RotaryEncoder_Alps_EC11E-Switch_Vertical_H20mm_CircularMountingHoles
- gave numbers to parts that had none: 1
Connections:
- wire segments 62 -> 70
- no-connect marks 0 -> 17

Commit message: PCB completed and schematic updated
Connections:
- wire segments 70 -> 72
- no-connect marks 17 -> 12
Other:
- moved on the sheet: U1
